Commit message: New all-in-one bringup launch file for base driver

File: omni_base_driver/urdf/omni.urdf (robot description, URDF)
Before this commit: robot omni_bot, 3 links, 2 joints
Links:
- removed link base_imu
- added link imu
Joints:
- joint base_link_to_imu: child base_imu -> imu; origin xyz=-0.005 0.035 -0.06 rpy=1.570796327 0.0 3.1415926 -> xyz=-0.005 0.035 -0.06 rpy=3.1415926 0.0 0.0
- joint base_link_to_laser: origin xyz=0.0 0.0 0.125 rpy=0.0 0.0 3.1415926 -> xyz=0.0 0.0 0.125 rpy=0.0 0.0 0.0
